File: base-shield/base-shield.kicad_pcb (KiCad board)
At the start: 2 copper layers, 101.6 x 53.3 mm, 14 parts, among them J1 Barrel_Jack_Switch, J2 Conn_01x02, P1 Digital, P10 CONN_01X01, P11 CONN_01X01, P13 CONN_01X01, P2 Power, P3 Analog, P4 Analog, P5 PWM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

Commit message: aaa
Parts:
- added D1: LED, LED_THT:LED_D3.0mm_Clear, F.Cu at (108.5, 106.4)
- added Q1: 2N7000, Package_TO_SOT_THT:TO-126-3_Horizontal_TabDown, F.Cu at (144.0, 92.5)
- added R1: R, Resistor_THT:R_Axial_DIN0204_L3.6mm_D1.6mm_P5.08mm_Horizontal, F.Cu at (131.3, 106.4)
- added SW1: SW_Push, Button_Switch_THT:SW_PUSH_6mm, F.Cu at (128.1, 119.1)
- moved C1 2.54 mm to (131.3, 93.7)
Connections:
- J2 pad 1: Net-(C1-Pad1) -> Net-(J2-Pad1)
Routing:
- net /A0: track 0.00 -> 69.0 mm
- net Net-(C1-Pad1): track 18.3 -> 59.3 mm
- net Net-(J2-Pad1): track 0.00 -> 24.4 mm
- net Net-(D1-Pad1): track 0.00 -> 22.9 mm
- net GND: track 33.4 -> 53.5 mm
- net /Reset: track 0.00 -> 9.92 mm
Other:
- board size 101.6 x 53.3 mm -> 99.1 x 53.3 mm
