File: base-shield/base-shield.sch (KiCad schematic (older format))
At the start: 16 parts, among them J1 Barrel_Jack_Switch, J2 Conn_01x02, P1 Digital, P10 CONN_01X01, P11 CONN_01X01, P12 CONN_01X01, P13 CONN_01X01, P2 Power, P3 Analog, P4 Analog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

Commit message: aaa
Parts:
- added D1: LED, LED_THT:LED_D3.0mm_Clear, symbol Device:LED
- added Q1: 2N7000, Package_TO_SOT_THT:TO-126-3_Horizontal_TabDown, symbol Transistor_FET:2N7000
- added R1: R, Resistor_THT:R_Axial_DIN0204_L3.6mm_D1.6mm_P5.08mm_Horizontal, symbol Device:R
- added SW1: SW_Push, Button_Switch_THT:SW_PUSH_6mm, symbol Switch:SW_Push
Connections:
- net A0: now also D1.2 (A), Q1.2 (G)
- net GND: now also R1.2, SW1.2
- net Reset: now also SW1.1
- net at C1.1, J1.1: now also Q1.3 (D); no longer J2.1 (Pin_1)
- new net: J2.1 (Pin_1), Q1.1 (S)
- new net: D1.1 (K), R1.1
- no-connect marks 84 -> 82
Other:
- moved on the sheet: C1, J2
Changed lines of the file:
@@
 52(SCK)
 NoConn ~ 9250 1200
-NoConn ~ 8600 1550
 NoConn ~ 8900 1200
 Wire Wire Line
@@
 NoConn ~ 10400 4000
 NoConn ~ 10400 4100
-NoConn ~ 8900 2450
 NoConn ~ 8900 2550
 NoConn ~ 8900 2650
@@
 L Connector_Generic:Conn_01x02 J2
 U 1 1 5D5041B5
-P 5700 2400
-F 0 "J2" H 5780 2392 50  0000 L CNN
-F 1 "Conn_01x02" H 5780 2301 50  0000 L CNN
-F 2 "Connector_PinSocket_2.54mm:PinSocket_1x02_P2.54mm_Vertical" H 5700 2400 50  0001 C CNN
-F 3 "~" H 5700 2400 50  0001 C CNN
-	1    5700 2400
-	1    0    0    -1
-$EndComp
-$Comp
-L Device:C C1
-U 1 1 5D50514B
-P 5000 2550
-F 0 "C1" H 5115 2596 50  0000 L CNN
-F 1 "C" H 5115 2505 50  0000 L CNN
-F 2 "Capacitor_THT:CP_Radial_D5.0mm_P2.50mm" H 5038 2400 50  0001 C CNN
-F 3 "~" H 5000 2550 50  0001 C CNN
-	1    5000 2550
+P 6700 3450
+F 0 "J2" H 6780 3442 50  0000 L CNN
+F 1 "Conn_01x02" H 6780 3351 50  0000 L CNN
+F 2 "Connector_PinSocket_2.54mm:PinSocket_1x02_P2.54mm_Vertical" H 6700 3450 50  0001 C CNN
+F 3 "~" H 6700 3450 50  0001 C CNN
+	1    6700 3450
 	1    0    0    -1
 $EndComp
@@
 Wire Wire Line
 	4300 2600 4500 2600
-Wire Wire Line
-	4500 2600 4500 2700
 $Comp
 L power:GND #PWR07
 U 1 1 5D514379
-P 4500 3000
-F 0 "#PWR07" H 4500 2750 50  0001 C CNN
-F 1 "GND" H 4505 2827 50  0000 C CNN
-F 2 "" H 4500 3000 50  0001 C CNN
-F 3 "" H 4500 3000 50  0001 C CNN
-	1    4500 3000
-	1    0    0    -1
-$EndComp
+P 4500 3750
+F 0 "#PWR07" H 4500 3500 50  0001 C CNN
+F 1 "GND" H 4505 3577 50  0000 C CNN
+F 2 "" H 4500 3750 50  0001 C CNN
+F 3 "" H 4500 3750 50  0001 C CNN
+	1    4500 3750
+	1    0    0    -1
+$EndComp
+$Comp
+L Transistor_FET:2N7000 Q1
+U 1 1 5ED0ADE1
+P 6400 2750
+F 0 "Q1" V 6651 2750 50  0000 C CNN
+F 1 "2N7000" V 6742 2750 50  0000 C CNN
+F 2 "Package_TO_SOT_THT:TO-126-3_Horizontal_TabDown" H 6600 2675 50  0001 L CIN
+F 3 "https://www.fairchildsemi.com/datasheets/2N/2N7000.pdf" H 6400 2750 50  0001 L CNN
+	1    6400 2750
+	1    0    0    -1
+$EndComp
+Wire Wire Line
+	6500 2400 6500 2550
+Text Label 5500 2750 0    50   ~ 0
+A0
+Wire Wire Line
+	4500 3750 4500 3550
+Connection ~ 4500 3550
+Wire Wire Line
+	4500 2600 4500 3550
+Wire Wire Line
+	6500 2950 6500 3450
+$Comp
+L Device:R R1
+U 1 1 5ED4539B
+P 6000 3350
+F 0 "R1" H 6070 3396 50  0000 L CNN
+F 1 "R" H 6070 3305 50  0000 L CNN
+F 2 "Resistor_THT:R_Axial_DIN0204_L3.6mm_D1.6mm_P5.08mm_Horizontal" V 5930 3350 50  0001 C CNN
+F 3 "~" H 6000 3350 50  0001 C CNN
+	1    6000 3350
+	1    0    0    -1
+$EndComp
+$Comp
+L Device:C C1
+U 1 1 5D50514B
+P 5000 3000
+F 0 "C1" H 5115 3046 50  0000 L CNN
+F 1 "C" H 5115 2955 50  0000 L CNN
+F 2 "Capacitor_THT:CP_Radial_D5.0mm_P2.50mm" H 5038 2850 50  0001 C CNN
+F 3 "~" H 5000 3000 50  0001 C CNN
+	1    5000 3000
+	1    0    0    -1
+$EndComp
+Wire Wire Line
+	5000 2400 6500 2400
 Wire Wire Line
 	4300 2400 5000 2400
-Wire Wire Line
-	4500 2700 5000 2700
-Connection ~ 4500 2700
-Wire Wire Line
-	4500 2700 4500 3000
-Wire Wire Line
-	5000 2400 5500 2400
 Connection ~ 5000 2400
 Wire Wire Line
-	5000 2700 5500 2700
-Wire Wire Line
-	5500 2700 5500 2500
-Connection ~ 5000 2700
+	5000 2400 5000 2850
+Wire Wire Line
+	4500 3550 5000 3550
+Connection ~ 5000 3550
+Wire Wire Line
+	5000 3150 5000 3550
+Wire Wire Line
+	3300 3550 3800 3550
+Text Label 3300 3550 0    50   ~ 0
+Reset
+$Comp
+L Switch:SW_Push SW1
+U 1 1 5EDE050B
+P 4000 3550
+F 0 "SW1" H 4000 3835 50  0000 C CNN
+F 1 "SW_Push" H 4000 3744 50  0000 C CNN
+F 2 "Button_Switch_THT:SW_PUSH_6mm" H 4000 3750 50  0001 C CNN
+F 3 "~" H 4000 3750 50  0001 C CNN
+	1    4000 3550
+	1    0    0    -1
+$EndComp
+Wire Wire Line
+	4200 3550 4500 3550
+$Comp
+L Device:LED D1
+U 1 1 5EDEB9A4
+P 6000 2950
+F 0 "D1" V 6039 2833 50  0000 R CNN
+F 1 "LED" V 5948 2833 50  0000 R CNN
+F 2 "LED_THT:LED_D3.0mm_Clear" H 6000 2950 50  0001 C CNN
+F 3 "~" H 6000 2950 50  0001 C CNN
+	1    6000 2950
+	0    -1   -1   0
+$EndComp
+Wire Wire Line
+	5000 3550 6000 3550
+Wire Wire Line
+	6000 2750 6000 2800
+Connection ~ 6000 2750
+Wire Wire Line
+	6000 2750 6200 2750
+Wire Wire Line
+	6000 3100 6000 3200
+Wire Wire Line
+	6000 3500 6000 3550
+Connection ~ 6000 3550
+Wire Wire Line
+	6000 3550 6500 3550
+Wire Wire Line
+	5500 2750 6000 2750
 $EndSCHEMATC
