File: switcher-shield/switcher-shield.kicad_pcb (KiCad board)
At the start: 2 copper layers, 101.6 x 53.3 mm, 34 parts, among them IC1 TB6643KQ,8, IC2 TB6643KQ,8, IC3 TB6643KQ,8, IC4 TB6643KQ,8, J1 Conn_02x16_Odd_Even, J10 Conn_01x02, J11 Conn_02x03_Odd_Even, J12 Conn_01x02, J13 Conn_01x02, J14 Conn_02x03_Odd_Even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

Commit message: aaa
Other:
- board size 101.6 x 53.3 mm -> 99.1 x 53.3 mm
Changed lines of the file:
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@@
   (general
     (thickness 1.6)
-    (drawings 18)
+    (drawings 16)
     (tracks 411)
     (zones 0)
@@
       (viasonmask true)
       (mode 1)
-      (useauxorigin false)
+      (useauxorigin true)
       (hpglpennumber 1)
       (hpglpenspeed 20)
@@
       (psa4output false)
       (plotreference true)
-      (plotvalue true)
+      (plotvalue false)
       (plotinvisibletext false)
       (padsonsilk false)
@@
     )
   )
+  (gr_line (start 202.438 81.026) (end 202.438 120.396) (layer Edge.Cuts) (width 0.15))
   (gr_line (start 113.538 78.994) (end 113.538 110.998) (layer F.SilkS) (width 0.15))
   (gr_line (start 103.378 78.994) (end 113.538 78.994) (layer F.SilkS) (width 0.15))
@@
   (gr_line (start 202.438 121.666) (end 103.378 121.666) (angle 90) (layer Edge.Cuts) (width 0.15))
   (gr_line (start 202.438 120.396) (end 202.438 121.666) (angle 90) (layer Edge.Cuts) (width 0.15))
-  (gr_line (start 204.978 117.856) (end 202.438 120.396) (angle 90) (layer Edge.Cuts) (width 0.15))
-  (gr_line (start 204.978 83.566) (end 204.978 117.856) (angle 90) (layer Edge.Cuts) (width 0.15))
-  (gr_line (start 202.438 81.026) (end 204.978 83.566) (angle 90) (layer Edge.Cuts) (width 0.15))
   (gr_line (start 202.438 70.866) (end 202.438 81.026) (angle 90) (layer Edge.Cuts) (width 0.15))
   (gr_line (start 199.898 68.326) (end 202.438 70.866) (angle 90) (layer Edge.Cuts) (width 0.15))
